Commit message: update urdf and launch file

File: obot_description/description/sensors/lidar.xacro (robot description, xacro)
@@ -6,5 +6,9 @@
         <parent link="chassis_link"/>
         <child link="lidar_link"/>
+<<<<<<< HEAD
         <origin xyz="0.1 0 0.18" rpy="0 0 0"/>
+=======
+        <origin xyz="0.12 0 0.18" rpy="0 0 0"/>
+>>>>>>> b43d28c (update urdf and launch file)
         <axis xyz="0 0 0"/>
     </joint>
@@ -37,8 +41,15 @@
                 <scan>
                 <horizontal>
+<<<<<<< HEAD
                     <samples>720</samples>
                     <resolution>1</resolution>
                     <min_angle>${-pi/3}</min_angle>
                     <max_angle>${pi/3}</max_angle>
+=======
+                    <samples>360</samples>
+                    <resolution>1</resolution>
+                    <min_angle>${-pi/1.5}</min_angle>
+                    <max_angle>${pi/1.5}</max_angle>
+>>>>>>> b43d28c (update urdf and launch file)
                 </horizontal>
                 </scan>

File: obot_description/description/urdf_description.xacro (robot description, xacro)
@@ -20,12 +20,21 @@
     </material>
     <xacro:property name="slab_height" value="0.3"/>
+<<<<<<< HEAD
     <xacro:property name="rviz_visual" value="false"/>
     <xacro:property name="gazebo_visual" value="true"/>
+=======
+    <xacro:property name="gazebo_visual" value="true"/>
+>>>>>>> b43d28c (update urdf and launch file)
     <xacro:arg name="laser_visual" default="false"/>
     <xacro:arg name="imu_visual"   default="true"/>
     <xacro:arg name="sonar_visual"   default="false"/>
     <xacro:arg name="cam_visual"   default="false"/>
+<<<<<<< HEAD
     <xacro:include filename="$(find obot_description)/description/macros.xacro"/>
     <xacro:include filename="$(find obot_description)/description/controllers.xacro"/>
+=======
+    <xacro:include filename="$(find obot_description)/description/inertia_macros.xacro"/>
+    <xacro:include filename="$(find obot_description)/description/part_macros.xacro"/>
+>>>>>>> b43d28c (update urdf and launch file)
     <!-- BASE LINK -->
     <!-- <base joint/> -->
@@ -43,7 +52,13 @@
             <origin xyz="0 0 0" rpy="0 0 0"/>
             <geometry>
+<<<<<<< HEAD
                 <xacro:if value="${rviz_visual}">
                     <mesh filename="package://obot_description/meshes/chassis.stl"/>
                 </xacro:if>
+=======
+                <xacro:unless value="${gazebo_visual}">
+                    <mesh filename="package://obot_description/meshes/chassis.stl"/>
+                </xacro:unless>
+>>>>>>> b43d28c (update urdf and launch file)
                 <xacro:if value="${gazebo_visual}">
                     <mesh filename="$(find obot_description)/meshes/chassis.stl"/>
@@ -52,4 +67,5 @@
             <material name="orange"/>
         </visual>
+<<<<<<< HEAD
         <visual>
             <origin xyz="0 0 ${0.15+slab_height}" rpy="0 0 0"/>
@@ -64,4 +80,6 @@
             <material name="orange"/>
         </visual>
+=======
+>>>>>>> b43d28c (update urdf and launch file)
         <collision>
             <origin xyz="0 0 0.075" rpy="0 0 0"/>
@@ -70,4 +88,5 @@
             </geometry>
         </collision>
+<<<<<<< HEAD
         <collision>
             <origin xyz="0 0 ${0.15+slab_height+0.005}" rpy="0 0 0"/>
@@ -76,4 +95,6 @@
             </geometry>
         </collision>
+=======
+>>>>>>> b43d28c (update urdf and launch file)
         <xacro:inertial_cylinder mass="10" length="0.15" radius="0.2">
             <origin xyz="0 0 0.075" rpy="0 0 0"/>
@@ -84,4 +105,5 @@
     </gazebo>
     <!--  ########################### -->
+<<<<<<< HEAD
     <!-- SUPPORT LINK -->
     <joint name="support_joint" type="fixed">
@@ -103,4 +125,7 @@
     </gazebo>
     <!--  ########################### -->
+=======
+    <xacro:include filename="$(find obot_description)/description/add_slab_macros.xacro"/>
+>>>>>>> b43d28c (update urdf and launch file)
     <!-- LEFT WHEEL LINK FRAME -->
     <joint name="left_wheel_joint" type="continuous">
@@ -225,4 +250,8 @@
     </gazebo>
     <!-- ##################################### -->
+<<<<<<< HEAD
+=======
+    <xacro:include filename="$(find obot_description)/description/controllers.xacro"/>
+>>>>>>> b43d28c (update urdf and launch file)
     <xacro:include filename="$(find obot_description)/description/sensors/imu.xacro"/>
     <xacro:include filename="$(find obot_description)/description/sensors/lidar.xacro"/>

Commit message: update urdf and launch file

File: obot_description/description/sensors/lidar.xacro (robot description, xacro)
@@ -6,9 +6,5 @@
         <parent link="chassis_link"/>
         <child link="lidar_link"/>
-<<<<<<< HEAD
-        <origin xyz="0.1 0 0.18" rpy="0 0 0"/>
-=======
         <origin xyz="0.12 0 0.18" rpy="0 0 0"/>
->>>>>>> b43d28c (update urdf and launch file)
         <axis xyz="0 0 0"/>
     </joint>

File: obot_description/description/urdf_description.xacro (robot description, xacro)
@@ -20,21 +20,11 @@
     </material>
     <xacro:property name="slab_height" value="0.3"/>
-<<<<<<< HEAD
-    <xacro:property name="rviz_visual" value="false"/>
     <xacro:property name="gazebo_visual" value="true"/>
-=======
-    <xacro:property name="gazebo_visual" value="true"/>
->>>>>>> b43d28c (update urdf and launch file)
     <xacro:arg name="laser_visual" default="false"/>
     <xacro:arg name="imu_visual"   default="true"/>
     <xacro:arg name="sonar_visual"   default="false"/>
     <xacro:arg name="cam_visual"   default="false"/>
-<<<<<<< HEAD
-    <xacro:include filename="$(find obot_description)/description/macros.xacro"/>
-    <xacro:include filename="$(find obot_description)/description/controllers.xacro"/>
-=======
     <xacro:include filename="$(find obot_description)/description/inertia_macros.xacro"/>
     <xacro:include filename="$(find obot_description)/description/part_macros.xacro"/>
->>>>>>> b43d28c (update urdf and launch file)
     <!-- BASE LINK -->
     <!-- <base joint/> -->
@@ -52,13 +42,7 @@
             <origin xyz="0 0 0" rpy="0 0 0"/>
             <geometry>
-<<<<<<< HEAD
-                <xacro:if value="${rviz_visual}">
-                    <mesh filename="package://obot_description/meshes/chassis.stl"/>
-                </xacro:if>
-=======
                 <xacro:unless value="${gazebo_visual}">
                     <mesh filename="package://obot_description/meshes/chassis.stl"/>
                 </xacro:unless>
->>>>>>> b43d28c (update urdf and launch file)
                 <xacro:if value="${gazebo_visual}">
                     <mesh filename="$(find obot_description)/meshes/chassis.stl"/>
@@ -67,19 +51,4 @@
             <material name="orange"/>
         </visual>
-<<<<<<< HEAD
-        <visual>
-            <origin xyz="0 0 ${0.15+slab_height}" rpy="0 0 0"/>
-            <geometry>
-                <xacro:if value="${rviz_visual}">
-                    <mesh filename="package://obot_description/meshes/slab.stl"/>
-                </xacro:if>
-                <xacro:if value="${gazebo_visual}">
-                    <mesh filename="$(find obot_description)/meshes/slab.stl"/>
-                </xacro:if>
-            </geometry>
-            <material name="orange"/>
-        </visual>
-=======
->>>>>>> b43d28c (update urdf and launch file)
         <collision>
             <origin xyz="0 0 0.075" rpy="0 0 0"/>
@@ -88,13 +57,4 @@
             </geometry>
         </collision>
-<<<<<<< HEAD
-        <collision>
-            <origin xyz="0 0 ${0.15+slab_height+0.005}" rpy="0 0 0"/>
-            <geometry>
-                <cylinder radius="0.2" length="0.01"/>
-            </geometry>
-        </collision>
-=======
->>>>>>> b43d28c (update urdf and launch file)
         <xacro:inertial_cylinder mass="10" length="0.15" radius="0.2">
             <origin xyz="0 0 0.075" rpy="0 0 0"/>
@@ -105,27 +65,5 @@
     </gazebo>
     <!--  ########################### -->
-<<<<<<< HEAD
-    <!-- SUPPORT LINK -->
-    <joint name="support_joint" type="fixed">
-        <parent link="chassis_link"/>
-        <child link="support_link"/>
-        <origin xyz="0 0 0.15"/>
-    </joint>
-    <link name="support_link">
-        <xacro:insert_support x="0.04" y="-0.14"/>
-        <xacro:insert_support x="0.04" y="0.14"/>
-        <xacro:insert_support x="-0.12" y="0.08"/>
-        <xacro:insert_support x="-0.12" y="-0.08"/>
-        <xacro:inertial_cylinder mass="0.8" length="${slab_height}" radius="0.1">
-            <origin xyz="0 0 0.1" rpy="0 0 0"/>
-        </xacro:inertial_cylinder>
-    </link>
-    <gazebo reference="support_link">
-        <material>Gazebo/White</material>
-    </gazebo>
-    <!--  ########################### -->
-=======
     <xacro:include filename="$(find obot_description)/description/add_slab_macros.xacro"/>
->>>>>>> b43d28c (update urdf and launch file)
     <!-- LEFT WHEEL LINK FRAME -->
     <joint name="left_wheel_joint" type="continuous">
@@ -250,8 +188,5 @@
     </gazebo>
     <!-- ##################################### -->
-<<<<<<< HEAD
-=======
     <xacro:include filename="$(find obot_description)/description/controllers.xacro"/>
->>>>>>> b43d28c (update urdf and launch file)
     <xacro:include filename="$(find obot_description)/description/sensors/imu.xacro"/>
     <xacro:include filename="$(find obot_description)/description/sensors/lidar.xacro"/>
